Commit message: Improve Pick and Place

File: sapling_ws/src/domains/arm/piper_description/urdf/piper_description.xacro (robot description, xacro)
@@ -508,5 +508,5 @@
      <parent link="link6"/>
      <child link = "grasp_tcp"/>
-     <origin xyz="0 0 0.145" rpy = "0 0 0"/>
+     <origin xyz="0 0 0.072" rpy = "0 0 0"/>
   </joint>
 <!-- controller -->
