Commit message: NEWEST COMMIT AFTER URDF MERGE

File: sapling_ws/src/domains/arm/piper_description/urdf/piper_description.urdf (robot description, URDF)
Before this commit: robot piper, 10 links, 9 joints
Links:
- removed link base_link
- added link arm_base_link, mass 1.02; collision mesh filename=package://piper_description/meshes/base_link.STL; visual mesh filename=package://piper_description/meshes/base_link.STL
Joints:
- joint joint1: parent base_link -> arm_base_link

File: sapling_ws/src/domains/arm/piper_description/urdf/piper_description.xacro (robot description, xacro)
@@ -3,13 +3,7 @@
   name="piper"
   xmlns:xacro="http://ros.org/wiki/xacro">
-<!-- world -->
-  <link name="world"/>
-  <joint name="fixed_base_joint" type="fixed">
-      <parent link="world"/>
-      <child link="base_link"/>
-  </joint>
 <!-- arm -->
 <link
-    name="base_link">
+    name="arm_base_link">
     <inertial>
             <origin xyz="-0.00473641164191482 2.56829134630247E-05 0.041451518036016" rpy="0 0 0" />
@@ -79,5 +73,5 @@
       rpy="0 0 0" />
     <parent
-      link="base_link" />
+      link="arm_base_link" />
     <child
       link="link1" />

File: sapling_ws/src/domains/arm/piper_moveit/piper_with_gripper_moveit/config/piper.urdf.xacro (robot description, xacro)
@@ -1,7 +1,7 @@
 <?xml version="1.0"?>
-<robot xmlns:xacro="http://www.ros.org/wiki/xacro" name="piper">
+<robot xmlns:xacro="http://www.ros.org/wiki/xacro" name="sapling">
     <xacro:arg name="initial_positions_file" default="initial_positions.yaml" />
     <!-- Import piper urdf file -->
-    <xacro:include filename="$(find piper_description)/urdf/piper_description.xacro" />
+    <xacro:include filename="$(find sapling_description)/urdf/sapling_description.urdf.xacro" />
     <!-- Import control_xacro -->
     <xacro:include filename="piper.ros2_control.xacro" />
